File: RN2483shield.kicad_pcb (KiCad board)
At the start: 2 copper layers, 68.9 x 53.6 mm, 8 parts, among them J1 SCREW_TERMINAL, J2 SMA, J3 SMA, P1 CONN_01X06, P2 CONN_01X06, P3 CONN_01X06, U1 RN2483

Commit message: Cleaned up directory. Fixed libraries.
Parts:
- J1: footprint My_Library:JPM-SCREWTERMINAL-5MM-2 -> freetronics_footprints:SCREWTERMINAL-5MM-2
- moved J1 0.64 mm to (213.4, 88.3)
Connections:
- SHIELD1 pad 13: Net-(SHIELD1-Pad13) -> (no net)
- SHIELD1 pad 2: Net-(SHIELD1-Pad2) -> (no net)
- SHIELD1 pad 3: Net-(SHIELD1-Pad3) -> (no net)
- SHIELD1 pad 4: Net-(SHIELD1-Pad4) -> (no net)
- SHIELD1 pad 5: Net-(SHIELD1-Pad5) -> (no net)
- SHIELD1 pad 6: Net-(SHIELD1-Pad6) -> (no net)
- SHIELD1 pad 7: Net-(SHIELD1-Pad7) -> (no net)
- SHIELD1 pad AD0: Net-(SHIELD1-PadAD0) -> (no net)
- SHIELD1 pad AD1: Net-(SHIELD1-PadAD1) -> (no net)
- SHIELD1 pad AD2: Net-(SHIELD1-PadAD2) -> (no net)
- SHIELD1 pad AD3: Net-(SHIELD1-PadAD3) -> (no net)
- SHIELD1 pad AD4: Net-(SHIELD1-PadAD4) -> (no net)
- SHIELD1 pad AD5: Net-(SHIELD1-PadAD5) -> (no net)
- SHIELD1 pad AREF: Net-(SHIELD1-PadAREF) -> (no net)
- SHIELD1 pad IO_R: Net-(SHIELD1-PadIO_R) -> (no net)
- SHIELD1 pad NC: Net-(SHIELD1-PadNC) -> (no net)
- SHIELD1 pad RST: Net-(SHIELD1-PadRST) -> (no net)
- SHIELD1 pad SCL: Net-(SHIELD1-PadSCL) -> (no net)
- SHIELD1 pad SDA: Net-(SHIELD1-PadSDA) -> (no net)
- SHIELD1 pad SP1: Net-(SHIELD1-PadSP1) -> (no net)
- SHIELD1 pad SP2: Net-(SHIELD1-PadSP2) -> (no net)
- SHIELD1 pad SP3: Net-(SHIELD1-PadSP3) -> (no net)
- SHIELD1 pad SP4: Net-(SHIELD1-PadSP4) -> (no net)
- SHIELD1 pad SP5: Net-(SHIELD1-PadSP5) -> (no net)
- SHIELD1 pad SP6: Net-(SHIELD1-PadSP6) -> (no net)
- SHIELD1 pad V_IN: Net-(SHIELD1-PadV_IN) -> (no net)
- U1 pad 10: Net-(U1-Pad10) -> (no net)
- U1 pad 13: Net-(U1-Pad13) -> (no net)
- U1 pad 14: Net-(U1-Pad14) -> (no net)
- U1 pad 15: Net-(U1-Pad15) -> (no net)
- U1 pad 16: Net-(U1-Pad16) -> (no net)
- U1 pad 17: Net-(U1-Pad17) -> (no net)
- U1 pad 18: Net-(U1-Pad18) -> (no net)
- U1 pad 19: Net-(U1-Pad19) -> (no net)
- U1 pad 2: Net-(U1-Pad2) -> (no net)
- U1 pad 29: Net-(U1-Pad29) -> (no net)
- U1 pad 3: Net-(U1-Pad3) -> (no net)
- U1 pad 30: Net-(U1-Pad30) -> (no net)
- U1 pad 31: Net-(U1-Pad31) -> (no net)
- U1 pad 35: Net-(U1-Pad35) -> (no net)
- U1 pad 36: Net-(U1-Pad36) -> (no net)
- U1 pad 37: Net-(U1-Pad37) -> (no net)
- U1 pad 38: Net-(U1-Pad38) -> (no net)
- U1 pad 39: Net-(U1-Pad39) -> (no net)
- U1 pad 4: Net-(U1-Pad4) -> (no net)
- U1 pad 40: Net-(U1-Pad40) -> (no net)
- U1 pad 42: Net-(U1-Pad42) -> (no net)
- U1 pad 43: Net-(U1-Pad43) -> (no net)
- U1 pad 44: Net-(U1-Pad44) -> (no net)
- U1 pad 45: Net-(U1-Pad45) -> (no net)
- U1 pad 46: Net-(U1-Pad46) -> (no net)
- U1 pad 5: Net-(U1-Pad5) -> (no net)
- U1 pad 9: Net-(U1-Pad9) -> (no net)
Routing:
- net (no net): track 7.62 -> 8.94 mm
- net Net-(SHIELD1-Pad13): track 1.14 -> 0.00 mm

Commit message: More library include fixes. Polygon pour with thermal relief.
Parts:
- J2, J3: footprint My_Library:SMA_BOARD_UPRIGHT -> MyFootprints:SMA_BOARD_UPRIGHT
- U1: footprint My_Library:RN2483 -> MyFootprints:RN2483
