File: RN2483shield.sch (KiCad schematic (older format))
At the start: 8 parts, among them J1 SCREW_TERMINAL, J2 SMA, J3 SMA, P1 CONN_01X06, P2 CONN_01X06, P3 CONN_01X06, U1 RN2483

Commit message: Cleaned up directory. Fixed libraries.
Parts:
- J2, J3: footprint sma:SMA -> My_Library:SMA_BOARD_UPRIGHT
- U1: footprint MyFootprints:RN2483 -> My_Library:RN2483
Changed lines of the file:
@@
 EESchema Schematic File Version 2
-LIBS:freetronics_schematic
 LIBS:power
 LIBS:device
@@
 LIBS:valves
 LIBS:rn2483
+LIBS:freetronics_schematic
+LIBS:screw_terminal
 LIBS:sma_through
-LIBS:screw_terminal
 LIBS:sma
-LIBS:sma_edge
-LIBS:RN2483shield-cache
 EELAYER 25 0
 EELAYER END
@@
 F 0 "J2" H 8725 1515 60  0000 C CNN
 F 1 "SMA" H 8790 1440 60  0000 C CNN
-F 2 "sma:SMA" H 8775 1370 50  0000 C CNN
+F 2 "My_Library:SMA_BOARD_UPRIGHT" H 8775 1370 50  0000 C CNN
 F 3 "" H 8600 1200 60  0000 C CNN
 	1    8600 1200
@@
 F 0 "J3" H 7825 1515 60  0000 C CNN
 F 1 "SMA" H 7890 1440 60  0000 C CNN
-F 2 "sma:SMA" H 7875 1370 50  0000 C CNN
+F 2 "My_Library:SMA_BOARD_UPRIGHT" H 7875 1370 50  0000 C CNN
 F 3 "" H 7700 1200 60  0000 C CNN
 	1    7700 1200
@@
 F 0 "U1" H 8400 1750 60  0000 C CNN
 F 1 "RN2483" H 7800 1750 60  0000 C CNN
-F 2 "MyFootprints:RN2483" H 8300 2500 60  0001 C CNN
+F 2 "My_Library:RN2483" H 8300 2500 60  0001 C CNN
 F 3 "" H 8300 2500 60  0000 C CNN
 	1    8200 3200

Commit message: More library include fixes. Polygon pour with thermal relief.
Parts:
- J2, J3: footprint My_Library:SMA_BOARD_UPRIGHT -> MyFootprints:SMA_BOARD_UPRIGHT
- U1: footprint My_Library:RN2483 -> MyFootprints:RN2483
Changed lines of the file:
@@
 LIBS:sma_through
 LIBS:sma
+LIBS:RN2483shield-cache
 EELAYER 25 0
 EELAYER END
@@
 F 0 "J2" H 8725 1515 60  0000 C CNN
 F 1 "SMA" H 8790 1440 60  0000 C CNN
-F 2 "My_Library:SMA_BOARD_UPRIGHT" H 8775 1370 50  0000 C CNN
+F 2 "MyFootprints:SMA_BOARD_UPRIGHT" H 8775 1370 50  0000 C CNN
 F 3 "" H 8600 1200 60  0000 C CNN
 	1    8600 1200
@@
 F 0 "J3" H 7825 1515 60  0000 C CNN
 F 1 "SMA" H 7890 1440 60  0000 C CNN
-F 2 "My_Library:SMA_BOARD_UPRIGHT" H 7875 1370 50  0000 C CNN
+F 2 "MyFootprints:SMA_BOARD_UPRIGHT" H 7875 1370 50  0000 C CNN
 F 3 "" H 7700 1200 60  0000 C CNN
 	1    7700 1200
@@
 F 0 "U1" H 8400 1750 60  0000 C CNN
 F 1 "RN2483" H 7800 1750 60  0000 C CNN
-F 2 "My_Library:RN2483" H 8300 2500 60  0001 C CNN
+F 2 "MyFootprints:RN2483" H 8300 2500 60  0001 C CNN
 F 3 "" H 8300 2500 60  0000 C CNN
 	1    8200 3200
